File: QL_Miracle_Trump_RAM/QL_Miracle_Trump_RAM.kicad_pcb (KiCad board)
At the start: 2 copper layers, 122.6 x 97.8 mm, 30 parts, among them J1 QL_SLOT_DIN41612_FEMALE-90deg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, J2 QL_SLOT_DIN41612_MALE_90degre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, U1 L7805, U10 MB81256, U11 MB81256, U12 MB81256, U13 MB81256, U14 MB81256, U15 MB81256, U16 MB81256, U17 MB81256, U18 74LS257, U19 74LS257, U2 MB81256, U3 MB81256, U4 MB81256, U5 MB81256, U6 MB81256, U7 MB81256, U8 MB81256, U9 MB81256

Commit message: miracle card works
Parts:
- added D1: 1N4148, Diode_THT:D_DO-35_SOD27_P10.16mm_Horizontal, F.Cu at (197.8, 68.4)
- added JP1: Jumper_2_Bridged, Resistor_THT:R_Axial_DIN0207_L6.3mm_D2.5mm_P10.16mm_Horizontal, F.Cu at (197.8, 63.3)
- added JP2: Jumper_2_Bridged, Resistor_THT:R_Axial_DIN0207_L6.3mm_D2.5mm_P10.16mm_Horizontal, F.Cu at (187.7, 65.8)
- added U20: 74LS10, Package_DIP:DIP-14_W7.62mm, F.Cu at (174.3, 81.1)
- added U21: 74LS86, Package_DIP:DIP-14_W7.62mm, F.Cu at (194.0, 73.5)
- added U22: 74LS245, Package_DIP:DIP-20_W7.62mm, F.Cu at (195.3, 122.4)
- added U23: 4040, Package_DIP:DIP-16_W7.62mm, F.Cu at (173.7, 117.9)
Connections:
- J1 pad a2: /D3 -> /DQ3
- J1 pad a3: /D4 -> /DQ4
- J1 pad a4: /D5 -> /DQ5
- J1 pad a5: /D6 -> /DQ6
- J1 pad a6: /D7 -> /DQ7
- J1 pad b2: /D2 -> /DQ2
- J1 pad b3: /D1 -> /DQ1
- J1 pad b4: /D0 -> /DQ0
- U18 pad 10: /A11 -> /A1
- U18 pad 2: /A0 -> /A16
- U18 pad 3: /A8 -> /A14
- U18 pad 5: /A1 -> /A11
- U19 pad 13: /A14 -> /A0
Routing:
- net GND: track 175.5 -> 323.0 mm, vias 0 -> 1
- net VCC: track 148.0 -> 272.5 mm
- net /SP1: track 0.00 -> 107.6 mm, vias 0 -> 3
- net /RW: track 138.0 -> 212.6 mm
- net /A3: track 66.6 -> 116.5 mm
- net /A2: track 63.2 -> 107.9 mm
- net unconnected-(U21-Pad5): track 0.00 -> 44.5 mm
- net unconnected-(U21-Pad4): track 0.00 -> 41.3 mm
- net /DTACK: track 129.8 -> 169.2 mm, vias 1 -> 3
- net /DQ3: track 0.00 -> 36.5 mm
- net /A5: track 135.4 -> 170.2 mm
- net /A0: track 125.2 -> 158.8 mm
- net /D3: track 191.1 -> 158.0 mm
- net /MA8: track 33.0 -> 65.7 mm, vias 1 -> 2
- net /DQ4: track 0.00 -> 32.5 mm
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Other:
- board text added: "DERAM"
- board text added: "EXPAN"
- board text added: "Miracle"
- board text added: "Systems"
- board text removed: "EXPANDERAM"
- board text removed: "Miracle Systems"

Commit message: work on miracle
Parts:
- added C10: 100n, Capacitor_THT:C_Disc_D4.3mm_W1.9mm_P5.00mm, F.Cu at (171.8, 45.5)
- added C11: 100n, Capacitor_THT:C_Disc_D4.3mm_W1.9mm_P5.00mm, F.Cu at (171.8, 58.2)
- added C12: 100n, Capacitor_THT:C_Disc_D4.3mm_W1.9mm_P5.00mm, F.Cu at (156.6, 68.4)
- added C13: 100n, Capacitor_THT:C_Disc_D4.3mm_W1.9mm_P5.00mm, F.Cu at (156.6, 73.5)
- added C14: 100n, Capacitor_THT:C_Disc_D4.3mm_W1.9mm_P5.00mm, F.Cu at (150.8, 74.7)
- added C15: 100n, Capacitor_THT:C_Disc_D4.3mm_W1.9mm_P5.00mm, F.Cu at (151.1, 111.6)
- added C16: 100n, Capacitor_THT:C_Disc_D4.3mm_W1.9mm_P5.00mm, F.Cu at (149.2, 121.6)
- added D2: 1N4148, Diode_THT:D_DO-35_SOD27_P10.16mm_Horizontal, F.Cu at (169.9, 50.6)
- added D3: 1N4148, Diode_THT:D_DO-35_SOD27_P10.16mm_Horizontal, F.Cu at (169.9, 53.1)
- added D4: 1N4148, Diode_THT:D_DO-35_SOD27_P10.16mm_Horizontal, F.Cu at (177.5, 70.9)
- added D5: 1N4148, Diode_THT:D_DO-35_SOD27_P10.16mm_Horizontal, F.Cu at (154.7, 78.5)
- added D6: 1N4148, Diode_THT:D_DO-35_SOD27_P10.16mm_Horizontal, F.Cu at (163.5, 102.7)
- added D7: 1N4148, Diode_THT:D_DO-35_SOD27_P10.16mm_Horizontal, F.Cu at (163.5, 105.2)
- added R1: R, Resistor_THT:R_Axial_DIN0207_L6.3mm_D2.5mm_P10.16mm_Horizontal, F.Cu at (169.9, 48.1)
- added R10: 680, Resistor_THT:R_Axial_DIN0207_L6.3mm_D2.5mm_P10.16mm_Horizontal, F.Cu at (153.4, 112.8)
- added R11: 680, Resistor_THT:R_Axial_DIN0207_L6.3mm_D2.5mm_P10.16mm_Horizontal, F.Cu at (153.5, 115.4)
- added R12: 680, Resistor_THT:R_Axial_DIN0207_L6.3mm_D2.5mm_P10.16mm_Horizontal, F.Cu at (153.5, 117.9)
- added R13: 680, Resistor_THT:R_Axial_DIN0207_L6.3mm_D2.5mm_P10.16mm_Horizontal, F.Cu at (153.5, 120.3)
- added R14: 680, Resistor_THT:R_Axial_DIN0207_L6.3mm_D2.5mm_P10.16mm_Horizontal, F.Cu at (153.5, 122.9)
- added R15: 680, Resistor_THT:R_Axial_DIN0207_L6.3mm_D2.5mm_P10.16mm_Horizontal, F.Cu at (153.5, 125.3)
- added R2: R, Resistor_THT:R_Axial_DIN0207_L6.3mm_D2.5mm_P10.16mm_Horizontal, F.Cu at (169.9, 55.7)
- added R3: 47K 1%, Resistor_THT:R_Axial_DIN0207_L6.3mm_D2.5mm_P10.16mm_Horizontal, F.Cu at (154.7, 65.8)
- added R4: 240ohm 1%, Resistor_THT:R_Axial_DIN0207_L6.3mm_D2.5mm_P10.16mm_Horizontal, F.Cu at (154.7, 70.9)
- added R5: 2500ohm 1%, Resistor_THT:R_Axial_DIN0207_L6.3mm_D2.5mm_P10.16mm_Horizontal, F.Cu at (154.7, 76.0)
- added R6: 810ohm 1%, Resistor_THT:R_Axial_DIN0207_L6.3mm_D2.5mm_P10.16mm_Horizontal, F.Cu at (154.7, 81.1)
- added R7: 4K7, Resistor_THT:R_Axial_DIN0207_L6.3mm_D2.5mm_P10.16mm_Horizontal, F.Cu at (153.4, 100.1)
- added R8: 680, Resistor_THT:R_Axial_DIN0207_L6.3mm_D2.5mm_P10.16mm_Horizontal, F.Cu at (153.4, 107.8)
- added R9: 680, Resistor_THT:R_Axial_DIN0207_L6.3mm_D2.5mm_P10.16mm_Horizontal, F.Cu at (153.4, 110.3)
- added U24: 74LS257, Package_DIP:DIP-16_W7.62mm, F.Cu at (157.2, 60.8)
- added U25: 74LS00, Package_DIP:DIP-14_W7.62mm, F.Cu at (167.4, 58.2)
- C1: value 100u/25V -> 33u/16V
- C2, C5, C6, C7: value 100u/16V -> 22u/25V
- JP1: footprint Resistor_THT:R_Axial_DIN0207_L6.3mm_D2.5mm_P10.16mm_Horizontal -> 8bits:Jumper_P10.16mm_Horizontal
- JP2: value Jumper_2_Bridged -> Jumper_2_Opened; footprint Resistor_THT:R_Axial_DIN0207_L6.3mm_D2.5mm_P10.16mm_Horizontal -> 8bits:Jumper_P10.16mm_Horizontal
- moved U20 0.63 mm to (175.0, 81.1)
Connections:
- J2 pad a12: /RED -> unconnected-(J2-RED-Pada12)
- J2 pad a25: /DBG -> unconnected-(J2-~{DBG}-Pada25)
- J2 pad a26: /SP2 -> GND
- J2 pad a27: /DSMC -> /DSMC2
- J2 pad a28: /SP1 -> GND
- J2 pad a29: /SP0 -> GND
- J2 pad a30: /ma12v -> unconnected-(J2-+12V-Pada30)
- J2 pad a31: /me12v -> unconnected-(J2--12V-Pada31)
- J2 pad b10: /BR -> unconnected-(J2-~{BR}-Padb10)
- J2 pad b13: /CSYNC -> unconnected-(J2-~{CSYNC}-Padb13)
- J2 pad b14: /E -> unconnected-(J2-E-Padb14)
- J2 pad b15: /VSYNC -> unconnected-(J2-VSYNCH-Padb15)
- J2 pad b16: /VPA -> unconnected-(J2-~{VPA}-Padb16)
- J2 pad b17: /GREEN -> unconnected-(J2-GREEN-Padb17)
- J2 pad b18: /BLUE -> unconnected-(J2-BLUE-Padb18)
- J2 pad b19: /FC2 -> unconnected-(J2-FC2-Padb19)
- J2 pad b20: /FC1 -> unconnected-(J2-FC1-Padb20)
- J2 pad b21: /FC0 -> unconnected-(J2-FC0-Padb21)
- J2 pad b23: /ROMOE -> unconnected-(J2-ROMOEH-Padb23)
- J2 pad b26: /SP3 -> GND
- J2 pad b27: /IPL0 -> unconnected-(J2-~{IPLO}-Padb27)
- J2 pad b28: /BERR -> unconnected-(J2-~{BERR}-Padb28)
- J2 pad b29: /IPL1 -> unconnected-(J2-~{IPL1}-Padb29)
- J2 pad b9: /BG -> unconnected-(J2-~{BG}-Padb9)
- JP1 pad 2: /SP1 -> /DSMC2
- JP2 pad 1: /SP1 -> /DSMC2
- U10 pad 15: unconnected-(U10-~{CAS}-Pad15) -> /CAS
- U10 pad 3: unconnected-(U10-~{WR}-Pad3) -> /RW
- U10 pad 4: unconnected-(U10-~{RAS}-Pad4) -> /RAS2
- U11 pad 14: /D5 -> /D7
- U11 pad 15: unconnected-(U11-~{CAS}-Pad15) -> /CAS
- U11 pad 2: /D5 -> /D7
- U11 pad 3: unconnected-(U11-~{WR}-Pad3) -> /RW
- U11 pad 4: unconnected-(U11-~{RAS}-Pad4) -> /RAS2
- U12 pad 15: unconnected-(U12-~{CAS}-Pad15) -> /CAS
- U12 pad 3: unconnected-(U12-~{WR}-Pad3) -> /RW
- U12 pad 4: unconnected-(U12-~{RAS}-Pad4) -> /RAS2
- U13 pad 15: unconnected-(U13-~{CAS}-Pad15) -> /CAS
- U13 pad 3: unconnected-(U13-~{WR}-Pad3) -> /RW
- U13 pad 4: unconnected-(U13-~{RAS}-Pad4) -> /RAS2
- U14 pad 15: unconnected-(U14-~{CAS}-Pad15) -> /CAS
- U14 pad 3: unconnected-(U14-~{WR}-Pad3) -> /RW
- U14 pad 4: unconnected-(U14-~{RAS}-Pad4) -> /RAS2
- U15 pad 15: unconnected-(U15-~{CAS}-Pad15) -> /CAS
- U15 pad 3: unconnected-(U15-~{WR}-Pad3) -> /RW
- U15 pad 4: unconnected-(U15-~{RAS}-Pad4) -> /RAS2
- U16 pad 14: /D6 -> /D5
- U16 pad 15: unconnected-(U16-~{CAS}-Pad15) -> /CAS
- U16 pad 2: /D6 -> /D5
- U16 pad 3: unconnected-(U16-~{WR}-Pad3) -> /RW
- U16 pad 4: unconnected-(U16-~{RAS}-Pad4) -> /RAS2
- U17 pad 14: /D7 -> /D6
- U17 pad 15: unconnected-(U17-~{CAS}-Pad15) -> /CAS
- U17 pad 2: /D7 -> /D6
- U17 pad 3: unconnected-(U17-~{WR}-Pad3) -> /RW
- U17 pad 4: unconnected-(U17-~{RAS}-Pad4) -> /RAS2
- U18 pad 10: /A1 -> /A0
- U18 pad 11: /A3 -> /A6
- U18 pad 13: /A10 -> /A9
- U18 pad 14: /A2 -> /A13
- U18 pad 6: /A9 -> /A10
- U19 pad 10: /A15 -> /A1
- U19 pad 11: /A7 -> /A4
- U19 pad 13: /A0 -> /A8
- U19 pad 14: /A6 -> /A12
- U19 pad 2: /A4 -> /A17
- U19 pad 3: /A12 -> /A15
- U19 pad 5: /A5 -> /A7
- U19 pad 6: /A13 -> /A5
- U2 pad 15: unconnected-(U2-~{CAS}-Pad15) -> /CAS
- U2 pad 3: unconnected-(U2-~{WR}-Pad3) -> /RW
- U2 pad 4: unconnected-(U2-~{RAS}-Pad4) -> /RAS
- U20 pad 5: unconnected-(U20-Pad5) -> Net-(D4-K)
- U20 pad 8: unconnected-(U20-Pad8) -> Net-(D5-A)
- U20 pad 9: unconnected-(U20-Pad9) -> Net-(U20-Pad9)
- U21 pad 2: /SP1 -> /DSMC2
- U23 pad 11: unconnected-(U23-Reset-Pad11) -> GND
- U23 pad 12: unconnected-(U23-Q8-Pad12) -> Net-(U23-Q8)
- U23 pad 13: unconnected-(U23-Q7-Pad13) -> Net-(U23-Q7)
- U23 pad 14: unconnected-(U23-Q9-Pad14) -> Net-(U23-Q9)
- U23 pad 15: unconnected-(U23-Q10-Pad15) -> Net-(U23-Q10)
- U23 pad 2: unconnected-(U23-Q5-Pad2) -> Net-(U23-Q5)
- U23 pad 3: unconnected-(U23-Q4-Pad3) -> Net-(U23-Q4)
- U23 pad 4: unconnected-(U23-Q6-Pad4) -> Net-(U23-Q6)
- U23 pad 5: unconnected-(U23-Q3-Pad5) -> Net-(U23-Q3)
- U23 pad 9: unconnected-(U23-Q0-Pad9) -> Net-(U23-Q0)
- U3 pad 14: /D5 -> /D7
- U3 pad 15: unconnected-(U3-~{CAS}-Pad15) -> /CAS
- U3 pad 2: /D5 -> /D7
- U3 pad 3: unconnected-(U3-~{WR}-Pad3) -> /RW
- U3 pad 4: unconnected-(U3-~{RAS}-Pad4) -> /RAS
- U4 pad 15: unconnected-(U4-~{CAS}-Pad15) -> /CAS
- U4 pad 3: unconnected-(U4-~{WR}-Pad3) -> /RW
- U4 pad 4: unconnected-(U4-~{RAS}-Pad4) -> /RAS
- U5 pad 15: unconnected-(U5-~{CAS}-Pad15) -> /CAS
- U5 pad 3: unconnected-(U5-~{WR}-Pad3) -> /RW
- U5 pad 4: unconnected-(U5-~{RAS}-Pad4) -> /RAS
- U6 pad 15: unconnected-(U6-~{CAS}-Pad15) -> /CAS
- U6 pad 3: unconnected-(U6-~{WR}-Pad3) -> /RW
- U6 pad 4: unconnected-(U6-~{RAS}-Pad4) -> /RAS
- U7 pad 15: unconnected-(U7-~{CAS}-Pad15) -> /CAS
- U7 pad 3: unconnected-(U7-~{WR}-Pad3) -> /RW
- U7 pad 4: unconnected-(U7-~{RAS}-Pad4) -> /RAS
- U8 pad 14: /D6 -> /D5
- U8 pad 15: unconnected-(U8-~{CAS}-Pad15) -> /CAS
- U8 pad 2: /D6 -> /D5
- U8 pad 3: unconnected-(U8-~{WR}-Pad3) -> /RW
- U8 pad 4: unconnected-(U8-~{RAS}-Pad4) -> /RAS
- U9 pad 14: /D7 -> /D6
- U9 pad 15: unconnected-(U9-~{CAS}-Pad15) -> /CAS
- U9 pad 2: /D7 -> /D6
- U9 pad 3: unconnected-(U9-~{WR}-Pad3) -> /RW
- U9 pad 4: unconnected-(U9-~{RAS}-Pad4) -> /RAS
Routing:
- net VCC: track 272.5 -> 690.8 mm, vias 2 -> 6
- net GND: track 323.0 -> 566.2 mm
- net /RW: track 212.6 -> 413.1 mm
- net /CAS: track 0.00 -> 196.8 mm, vias 0 -> 3
- net /MA4: track 96.0 -> 258.9 mm
- net /MA1: track 88.7 -> 251.1 mm
- net /MA5: track 86.4 -> 248.7 mm
- net /MA8: track 65.7 -> 227.5 mm
- net /MA7: track 108.1 -> 267.7 mm
- net /MA3: track 91.9 -> 251.3 mm
- net /MA2: track 87.5 -> 246.3 mm
- net /MA6: track 100.5 -> 257.7 mm
- net /MA0: track 100.1 -> 235.7 mm
- net /RAS2: track 0.00 -> 118.1 mm
- net /D5: track 106.3 -> 218.1 mm, vias 0 -> 1
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Other:
- board text added: "2026 - Repro by Alvaro A."
- board text removed: "(C) 2022-2026 Alvaro Alea Fdz"
- board text removed: "By Alvaro Alea Fdz."
- board text removed: "JLCJLCJLCJLC"
- board text removed: "REV.3"
- board text removed: "SINCLAIR QL 896kB RAM"
- board text removed: "www.va-de-retro.com"

Commit message: Miracle RAM probably finished
Parts:
- removed the C1 at (199.7, 59.5)
- removed the C2 at (133.8, 43.0)
- removed the C5 at (110.9, 43.0)
- removed the C6 at (133.8, 129.3)
- added C12: 22u/25V, Capacitor_THT:CP_Radial_D8.0mm_P5.00mm, F.Cu at (133.7, 43.0)
- added C13: 22u/25V, Capacitor_THT:CP_Radial_D8.0mm_P5.00mm, F.Cu at (110.9, 43.0)
- added C14: 22u/25V, Capacitor_THT:CP_Radial_D8.0mm_P5.00mm, F.Cu at (133.7, 129.3)
- added C15: 33u/16V, Capacitor_THT:CP_Axial_L11.0mm_D5.0mm_P18.00mm_Horizontal, F.Cu at (199.7, 59.5)
- C1: renamed from C13; value 100n -> 10n
- C2: renamed from C12; value 100n -> 10n
- C3: renamed from C14; value 100n -> 10n
- C4: renamed from C15; value 100n -> 10n
- C5: renamed from C11; value 100n -> 10n
- C6: renamed from C10; value 100n -> 10n
- R10: renamed from R6; value 810ohm 1% -> 820 1%
- R11: renamed from R5; value 2500ohm 1% -> 3K6 1%
- R12: renamed from R4; value 240ohm 1% -> 240 1%
- R13: renamed from R3; value 47K 1% -> 470 1%
- R15: renamed from R2; value R -> 5K6
- R16: renamed from R1; value R -> 3K3
- renumbered C3 to C10, C4 to C11, D7 to D1, D6 to D2, D5 to D3, D1 to D5, D3 to D7, D2 to D8, JP1 to JP-D6, JP2 to JP-R14, R15 to R1, R14 to R2, R13 to R3, R12 to R4, R11 to R5, R10 to R6, R9 to R7, R7 to R9
Connections:
- C1 pad 1: Net-(U24-I0b) -> Net-(D3-K)
- C1 pad 2: unconnected-(C13-Pad2) -> GND
- C2 pad 1: Net-(C12-Pad1) -> Net-(C2-Pad1)
- C3 pad 1: unconnected-(C14-Pad1) -> GND
- C4 pad 1: Net-(C15-Pad1) -> Net-(U18-S)
- C5 pad 1: Net-(D3-K) -> Net-(D7-K)
- D1 pad 1: unconnected-(D7-K-Pad1) -> Net-(D1-K)
- D1 pad 2: Net-(D6-A) -> Net-(D1-A)
- D2 pad 1: unconnected-(D6-K-Pad1) -> Net-(D2-K)
- D2 pad 2: Net-(D6-A) -> Net-(D1-A)
- D3 pad 1: unconnected-(D5-K-Pad1) -> Net-(D3-K)
- D3 pad 2: Net-(D5-A) (its old number) -> Net-(D3-A)
- D4 pad 1: Net-(D4-K) -> /CAS
- D4 pad 2: unconnected-(D4-A-Pad2) -> /DTACK
- D7 pad 1: Net-(D3-K) -> Net-(D7-K)
- D7 pad 2: Net-(D2-A) -> Net-(D7-A)
- D8 pad 2: Net-(D2-A) -> Net-(D7-A)
- R10 pad 1: Net-(C15-Pad1) -> Net-(U18-S)
- R10 pad 2: Net-(D5-A) (its old number) -> Net-(D3-A)
- R11 pad 1: Net-(U24-I0b) -> Net-(D3-K)
- R11 pad 2: unconnected-(R5-Pad2) -> GND
- R12 pad 2: Net-(D5-A) (its old number) -> Net-(D3-A)
- R13 pad 1: Net-(C12-Pad1) -> Net-(C2-Pad1)
- R15 pad 1: Net-(D3-K) -> Net-(D7-K)
- R9 pad 1: Net-(D6-A) -> Net-(D1-A)
- U18 pad 15: Net-(U18-OE) -> Net-(D3-A)
- U19 pad 15: Net-(U18-OE) -> Net-(D3-A)
- U20 pad 10: unconnected-(U20-Pad10) -> Net-(U23-CLK)
- U20 pad 12: unconnected-(U20-Pad12) -> /DIR245
- U20 pad 13: unconnected-(U20-Pad13) -> Net-(U20-Pad13)
- U20 pad 2: Net-(U20-Pad2) -> Net-(U23-CLK)
- U20 pad 4: unconnected-(U20-Pad4) -> Net-(U20-Pad3)
- U20 pad 5: Net-(D4-K) -> /CAS
- U20 pad 6: unconnected-(U20-Pad6) -> Net-(U20-Pad13)
- U20 pad 8: Net-(D5-A) (its old number) -> Net-(D3-A)
- U21 pad 10: unconnected-(U21-Pad10) -> Net-(C2-Pad1)
- U21 pad 11: Net-(U20-Pad2) -> Net-(U23-CLK)
- U21 pad 13: unconnected-(U21-Pad13) -> VCC
- U21 pad 4: unconnected-(U21-Pad4) -> /A18
- U21 pad 5: unconnected-(U21-Pad5) -> /A19
- U21 pad 9: unconnected-(U21-Pad9) -> GND
- U22 pad 1: /RW -> /DIR245
- U23 pad 10: unconnected-(U23-CLK-Pad10) -> Net-(U23-CLK)
- U23 pad 6: unconnected-(U23-Q2-Pad6) -> Net-(D1-K)
- U23 pad 7: unconnected-(U23-Q1-Pad7) -> Net-(D2-K)
- U24 pad 11: unconnected-(U24-I0d-Pad11) -> /A19
- U24 pad 14: unconnected-(U24-I0c-Pad14) -> /A18
- U24 pad 5: Net-(U24-I0b) -> Net-(D3-K)
- U24 pad 7: Net-(D4-K) -> /CAS
- U25 pad 1: unconnected-(U25-Pad1) -> Net-(U23-CLK)
- U25 pad 10: Net-(U25-Pad10) -> Net-(D7-A)
- U25 pad 12: unconnected-(U25-Pad12) -> Net-(D7-K)
- U25 pad 13: unconnected-(U25-Pad13) -> Net-(D1-A)
- U25 pad 2: unconnected-(U25-Pad2) -> Net-(D1-A)
- U25 pad 3: Net-(D2-A) -> Net-(D7-A)
- U25 pad 6: unconnected-(U25-Pad6) -> Net-(U24-I1c)
- U25 pad 9: Net-(U25-Pad10) -> Net-(D7-A)
Routing:
- net /DIR245: track 0.00 -> 119.1 mm, vias 0 -> 1
- net Net-(D3-A): track 0.00 -> 95.0 mm
- net Net-(U23-CLK): track 0.00 -> 93.3 mm, vias 0 -> 1
- net Net-(U18-S): track 11.4 -> 95.5 mm, vias 0 -> 1
- net Net-(D1-A): track 0.00 -> 80.1 mm, vias 0 -> 1
- net /A19: track 162.6 -> 235.0 mm, vias 1 -> 3
- net /A18: track 153.7 -> 213.3 mm
- net GND: track 566.2 -> 623.1 mm, vias 1 -> 2
- net Net-(C2-Pad1): track 0.00 -> 55.9 mm, vias 0 -> 4
- net unconnected-(U20-Pad12): track 50.9 -> 0.00 mm, vias 1 -> 0
- net Net-(C15-Pad1): track 49.4 -> 0.00 mm, vias 1 -> 0
- net Net-(D6-A): track 48.8 -> 0.00 mm
- net Net-(U20-Pad2): track 48.5 -> 0.00 mm
- net /RW: track 413.1 -> 365.5 mm
- net /CAS: track 196.8 -> 243.9 mm
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