File: QL_Miracle_Trump_RAM/QL_Miracle_Trump_RAM.kicad_sch (KiCad schematic)
At the start: 30 parts, among them J1 QL_SLOT_DIN41612_FEMALE-90deg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, J2 QL_SLOT_DIN41612_MALE_90degre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, U1 L7805, U10 MB81256, U11 MB81256, U12 MB81256, U13 MB81256, U14 MB81256, U15 MB81256, U16 MB81256, U17 MB81256, U18 74LS257, U19 74LS257, U2 MB81256, U3 MB81256, U4 MB81256, U5 MB81256, U6 MB81256, U7 MB81256, U8 MB81256, U9 MB81256

Commit message: miracle card works
Parts:
- added D1: 1N4148, Diode_THT:D_DO-35_SOD27_P10.16mm_Horizontal, symbol Diode:1N4148
- added JP1, JP2: Jumper_2_Bridged, Resistor_THT:R_Axial_DIN0207_L6.3mm_D2.5mm_P10.16mm_Horizontal, symbol Jumper:Jumper_2_Bridged
- added U20: 74LS10, Package_DIP:DIP-14_W7.62mm, symbol 74xx:74LS10
- added U21: 74LS86, Package_DIP:DIP-14_W7.62mm, symbol 74xx:74LS86
- added U22: 74LS245, Package_DIP:DIP-20_W7.62mm, symbol 74xx:74LS245
- added U23: 4040, Package_DIP:DIP-16_W7.62mm, symbol 4xxx:4040
Connections:
- net A0: now also U19.13 (I1c); no longer U18.2 (I0a)
- net A1: now also U18.10 (I1d); no longer U18.5 (I0b)
- net A11: now also U18.5 (I0b); no longer U18.10 (I1d)
- net A14: now also U18.3 (I1a); no longer U19.13 (I1c)
- net A16: now also U18.2 (I0a)
- net A8: no longer U18.3 (I1a)
- net D0: now also U22.16 (B2); no longer J1.b4 (D0)
- net D1: now also U22.14 (B4); no longer J1.b3 (D1)
- net D2: now also U22.12 (B6); no longer J1.b2 (D2)
- net D3: now also U22.11 (B7); no longer J1.a2 (D3)
- net D4: now also U22.13 (B5); no longer J1.a3 (D4)
- net D5: now also U22.15 (B3); no longer J1.a4 (D5)
- net D6: now also U22.17 (B1); no longer J1.a5 (D6)
- net D7: now also U22.18 (B0); no longer J1.a6 (D7)
- net DS: now also U21.12
- net DSMC: now also D1.1 (K), JP1.1 (A)
- net GND: now also JP2.2 (B), U20.7 (GND), U21.7 (GND), U22.10 (GND), U22.19 (CE), U23.8 (VSS)
- net MA8: now also U21.8
- net RW: now also U20.1, U22.1 (A->B)
- net SP1: now also JP1.2 (B), JP2.1 (A), U21.2
- net VCC: now also U20.14 (VCC), U21.1, U21.14 (VCC), U22.20 (VCC), U23.16 (VDD)
- new net: D1.2 (A), U20.11, U21.6
- new net: U20.3, U21.3
- new net: U20.2, U21.11
- new net DQ0: J1.b4 (D0), U22.4 (A2)
- new net DQ1: J1.b3 (D1), U22.6 (A4)
- new net DQ2: J1.b2 (D2), U22.8 (A6)
- new net DQ3: J1.a2 (D3), U22.9 (A7)
- new net DQ4: J1.a3 (D4), U22.7 (A5)
- new net DQ5: J1.a4 (D5), U22.5 (A3)
- new net DQ6: J1.a5 (D6), U22.3 (A1)
- new net DQ7: J1.a6 (D7), U22.2 (A0)
Other:
- moved on the sheet: J2, U10, U11, U12, U13, U14, U15, U16, U17, U18, U19, U2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

Commit message: work on miracle
Parts:
- added C10, C11, C12, C13, C14, C15, C16: 100n, Capacitor_THT:C_Disc_D4.3mm_W1.9mm_P5.00mm, symbol Device:C
- added D2, D3, D4, D5, D6, D7: 1N4148, Diode_THT:D_DO-35_SOD27_P10.16mm_Horizontal, symbol Diode:1N4148
- added R1, R2: R, Resistor_THT:R_Axial_DIN0207_L6.3mm_D2.5mm_P10.16mm_Horizontal, symbol Device:R
- added R10, R11, R12, R13, R14, R15, R8, R9: 680, Resistor_THT:R_Axial_DIN0207_L6.3mm_D2.5mm_P10.16mm_Horizontal, symbol Device:R
- added R3: 47K 1%, Resistor_THT:R_Axial_DIN0207_L6.3mm_D2.5mm_P10.16mm_Horizontal, symbol Device:R
- added R4: 240ohm 1%, Resistor_THT:R_Axial_DIN0207_L6.3mm_D2.5mm_P10.16mm_Horizontal, symbol Device:R
- added R5: 2500ohm 1%, Resistor_THT:R_Axial_DIN0207_L6.3mm_D2.5mm_P10.16mm_Horizontal, symbol Device:R
- added R6: 810ohm 1%, Resistor_THT:R_Axial_DIN0207_L6.3mm_D2.5mm_P10.16mm_Horizontal, symbol Device:R
- added R7: 4K7, Resistor_THT:R_Axial_DIN0207_L6.3mm_D2.5mm_P10.16mm_Horizontal, symbol Device:R
- added U24: 74LS257, Package_DIP:DIP-16_W7.62mm, symbol 74xx:74LS257
- added U25: 74LS00, Package_DIP:DIP-14_W7.62mm, symbol 74xx:74LS00
- C1: value 100u/25V -> 33u/16V
- C2, C5, C6, C7: value 100u/16V -> 22u/25V
- JP1: footprint Resistor_THT:R_Axial_DIN0207_L6.3mm_D2.5mm_P10.16mm_Horizontal -> 8bits:Jumper_P10.16mm_Horizontal
- JP2: value Jumper_2_Bridged -> Jumper_2_Opened; footprint Resistor_THT:R_Axial_DIN0207_L6.3mm_D2.5mm_P10.16mm_Horizontal -> 8bits:Jumper_P10.16mm_Horizontal; symbol Jumper:Jumper_2_Bridged -> Jumper:Jumper_2_Open
Connections:
- net A0: now also U18.10 (I1d); no longer U19.13 (I1c)
- net A1: now also U19.10 (I1d); no longer U18.10 (I1d)
- net A10: now also U18.6 (I1b); no longer U18.13 (I1c)
- net A12: now also U19.14 (I0c); no longer U19.3 (I1a)
- net A13: now also U18.14 (I0c); no longer U19.6 (I1b)
- net A15: now also U19.3 (I1a); no longer U19.10 (I1d)
- net A17: now also U19.2 (I0a)
- net A2: now also U24.3 (I1a); no longer U18.14 (I0c)
- net A3: now also U24.2 (I0a); no longer U18.11 (I0d)
- net A4: now also U19.11 (I0d); no longer U19.2 (I0a)
- net A5: now also U19.6 (I1b); no longer U19.5 (I0b)
- net A6: now also U18.11 (I0d); no longer U19.14 (I0c)
- net A7: now also U19.5 (I0b); no longer U19.11 (I0d)
- net A8: now also U19.13 (I1c)
- net A9: now also U18.13 (I1c); no longer U18.6 (I1b)
- net BERR: no longer J2.b28 (~{BERR})
- net BG: no longer J2.b9 (~{BG})
- net BLUE: no longer J2.b18 (BLUE)
- net BR: no longer J2.b10 (~{BR})
- net CSYNC: no longer J2.b13 (~{CSYNC})
- net D5: now also U16.14 (Q), U16.2 (D), U8.14 (Q), U8.2 (D); no longer U11.14 (Q), U11.2 (D), U3.14 (Q), U3.2 (D)
- net D6: now also U17.14 (Q), U17.2 (D), U9.14 (Q), U9.2 (D); no longer U16.14 (Q), U16.2 (D), U8.14 (Q), U8.2 (D)
- net D7: now also U11.14 (Q), U11.2 (D), U3.14 (Q), U3.2 (D); no longer U17.14 (Q), U17.2 (D), U9.14 (Q), U9.2 (D)
- net DBG: no longer J2.a25 (~{DBG})
- net DSMC: no longer J2.a27 (~{DSMC})
- net E: no longer J2.b14 (E)
- net FC0: no longer J2.b21 (FC0)
- net FC1: no longer J2.b20 (FC1)
- net FC2: no longer J2.b19 (FC2)
- net GND: now also J2.a26 (SP2), J2.a28 (SP1), J2.a29 (SP0), J2.b26 (SP3), U23.11 (Reset), C10.2, C11.2, C12.2, C15.2, C16.2, R1.2, R2.2, U24.15 (OE), U24.8 (GND), U25.7 (GND)
- net GREEN: no longer J2.b17 (GREEN)
- net IPL0: no longer J2.b27 (~{IPLO})
- net IPL1: no longer J2.b29 (~{IPL1})
- net MA0: now also R8.1
- net MA1: now also R9.1
- net MA2: now also R10.1
- net MA3: now also R14.1
- net MA4: now also R13.1
- net MA5: now also R12.1
- net MA6: now also R15.1
- net MA7: now also R11.1
- net RED: no longer J2.a12 (RED)
- net ROMOE: no longer J2.b23 (ROMOEH)
- net RW: now also U10.3 (~{WR}), U11.3 (~{WR}), U12.3 (~{WR}), U13.3 (~{WR}), U14.3 (~{WR}), U15.3 (~{WR}), U16.3 (~{WR}), U17.3 (~{WR}), U2.3 (~{WR}), U3.3 (~{WR}), U4.3 (~{WR}), U5.3 (~{WR}), U6.3 (~{WR}), U7.3 (~{WR}), U8.3 (~{WR}), U9.3 (~{WR})
- net SP0: no longer J2.a29 (SP0)
- net SP1: no longer J2.a28 (SP1), JP1.2 (B), JP2.1 (A), U21.2
- net SP2: no longer J2.a26 (SP2)
- net SP3: no longer J2.b26 (SP3)
- net VCC: now also C16.1, U24.16 (VCC), U24.6 (I1b), U25.14 (VCC)
- net VPA: no longer J2.b16 (~{VPA})
- net VSYNC: no longer J2.b15 (VSYNCH)
- net ma12v: no longer J2.a30 (+12V)
- net me12v: no longer J2.a31 (-12V)
- net CAS: now reaches U14.15 (~{CAS})
- net CAS: now also U10.15 (~{CAS}), U11.15 (~{CAS}), U12.15 (~{CAS}), U13.15 (~{CAS}), U15.15 (~{CAS}), U16.15 (~{CAS}), U17.15 (~{CAS}), U2.15 (~{CAS}), U3.15 (~{CAS}), U4.15 (~{CAS}), U5.15 (~{CAS}), U6.15 (~{CAS}), U7.15 (~{CAS}), U8.15 (~{CAS}), U9.15 (~{CAS})
- net RAS2: now reaches U14.4 (~{RAS})
- net RAS2: now also U10.4 (~{RAS}), U11.4 (~{RAS}), U12.4 (~{RAS}), U13.4 (~{RAS}), U15.4 (~{RAS}), U16.4 (~{RAS}), U17.4 (~{RAS}), U24.12 (Zc)
- net RAS: now reaches U8.4 (~{RAS})
- net RAS: now also U2.4 (~{RAS}), U3.4 (~{RAS}), U4.4 (~{RAS}), U5.4 (~{RAS}), U6.4 (~{RAS}), U7.4 (~{RAS}), U9.4 (~{RAS}), U24.9 (Zd)
- net at U20.8: now also D5.2 (A), R4.2, R6.2
- net at U20.9: now also U25.11
- net at U20.5: now also D4.1 (K), U24.7 (Zb)
- net at U23.12 (Q8): now also R8.2
- net at U23.13 (Q7): now also R9.2
- net at U23.14 (Q9): now also R10.2
- net at U23.15 (Q10): now also R11.2
- net at U23.2 (Q5): now also R15.2
- net at U23.3 (Q4): now also R14.2
- net at U23.4 (Q6): now also R13.2
- net at U23.5 (Q3): now also R12.2
- net at U23.9 (Q0): now also R7.2
- new net: C12.1, R3.1
- new net: C15.1, R6.1
- new net: C14.2, R4.1, U24.1 (S)
- new net: U24.10 (I1d), U24.13 (I1c)
- new net: R3.2, U24.4 (Za)
- new net: C13.1, R5.1, U24.5 (I0b)
- new net: D6.2 (A), D7.2 (A), R7.1
- new net: C11.1, D3.1 (K), R2.1
- new net: D2.2 (A), D3.2 (A), U25.3
- new net: U25.10, U25.9
- new net: U25.5, U25.8
- new net DEL1: C10.1, D2.1 (K), R1.1, U25.4
- new net DSMC2: J2.a27 (~{DSMC}), JP1.2 (B), JP2.1 (A), U21.2
- no-connect marks 0 -> 18
Other:
- company: (C) 2022 Alvaro Alea Fdz -> (C) 2026 Alvaro Alea Fdz
- title: External Expansion 512Kb memory for Sinclair QL -> Miracle ExpandRam 512Kb for Sinclair QL
- moved on the sheet: C1, C2, C3, C4, C5, C6, C7, C8, C9, D1, JP1, JP2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

Commit message: Miracle RAM probably finished
Parts:
- C1: renamed from C13; value 100n -> 10n
- C2: renamed from C12; value 100n -> 10n
- C3: renamed from C14; value 100n -> 10n
- C4: renamed from C15; value 100n -> 10n
- C5: renamed from C11; value 100n -> 10n
- C6: renamed from C10; value 100n -> 10n
- R10: renamed from R6; value 810ohm 1% -> 820 1%
- R11: renamed from R5; value 2500ohm 1% -> 3K6 1%
- R12: renamed from R4; value 240ohm 1% -> 240 1%
- R13: renamed from R3; value 47K 1% -> 470 1%
- R15: renamed from R2; value R -> 5K6
- R16: renamed from R1; value R -> 3K3
- renumbered C3 to C10, C4 to C11, C2 to C12, C5 to C13, C6 to C14, C1 to C15, D7 to D1, D6 to D2, D5 to D3, D1 to D5, D3 to D7, D2 to D8, JP1 to JP-D6, JP2 to JP-R14, R15 to R1, R14 to R2, R13 to R3, R12 to R4, R11 to R5, R10 to R6, R9 to R7, R7 to R9
Connections:
- net A18: now also U21.4, U24.14 (I0c)
- net A19: now also U21.5, U24.11 (I0d)
- net CAS: now also D4.1 (K), U20.5, U24.7 (Zb)
- net DTACK: now also D4.2 (A)
- net GND: now also C1.2, C3.1, R11.2, U21.9
- net RW: no longer U22.1 (A->B)
- net VCC: now also U21.13
- net at C2.1, R13.1: now also U21.10
- net at D3.1 (K): now also C1.1, R11.1, U24.5 (I0b)
- net at D3.2 (A), R10.2, R12.2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: now also U18.15 (OE), U19.15 (OE)
- net at U20.10: now also U20.2, U21.11, U23.10 (CLK), U25.1
- net at C4.1, R10.1: now also U18.1 (S), U19.1 (S)
- net at U20.3, U21.3: now also U20.4
- net at U20.6: now also U20.13
- net at U24.10 (I1d), U24.13 (I1c): now also U25.6
- net at D1.2 (A), D2.2 (A), R9.1: now also U25.13, U25.2
- net at C5.1, D7.1 (K), R15.1: now also U25.12
- net at D7.2 (A), D8.2 (A), U25.3: now also U25.10, U25.9
- net DIR245: now reaches U20.12
- net DIR245: now also U22.1 (A->B)
- net at D1.1 (K): now also U23.6 (Q2)
- net at D2.1 (K): now also U23.7 (Q1)
- no-connect marks 18 -> 19
Other:
- moved on the sheet: C1, C2, C3, C4, C5, C6, D1, D2, D3, D4, D5, D7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
